Commit message: Update urdf file

File: rebel_arm_description/urdf/arm.urdf (robot description, URDF)
Before this commit: robot arm, 8 links, 7 joints
Links:
- link link_0: geometry collision mesh filename=file://$(find rebel_arm_description)/meshes/link_0.stl scale=0.001 0.001 0.001; visual mesh filename=file://$(find rebel_arm_description)/meshes/link_0.dae scale=0.001 0.001 0.001
- link link_1: geometry collision mesh filename=file://$(find rebel_arm_description)/meshes/link_1.stl scale=0.001 0.001 0.001; visual mesh filename=file://$(find rebel_arm_description)/meshes/link_1.dae scale=0.001 0.001 0.001
- link link_2: geometry collision mesh filename=file://$(find rebel_arm_description)/meshes/link_2.stl scale=0.001 0.001 0.001; visual mesh filename=file://$(find rebel_arm_description)/meshes/link_2.dae scale=0.001 0.001 0.001
- link link_3: geometry collision mesh filename=file://$(find rebel_arm_description)/meshes/link_3.stl scale=0.001 0.001 0.001; visual mesh filename=file://$(find rebel_arm_description)/meshes/link_3.dae scale=0.001 0.001 0.001
- link link_4: geometry collision mesh filename=file://$(find rebel_arm_description)/meshes/link_4.stl scale=0.001 0.001 0.001; visual mesh filename=file://$(find rebel_arm_description)/meshes/link_4.dae scale=0.001 0.001 0.001
- link link_5: geometry collision mesh filename=file://$(find rebel_arm_description)/meshes/link_5.stl scale=0.001 0.001 0.001; visual mesh filename=file://$(find rebel_arm_description)/meshes/link_5.dae scale=0.001 0.001 0.001
- link link_6: geometry collision mesh filename=file://$(find rebel_arm_description)/meshes/link_6.stl scale=0.001 0.001 0.001; visual mesh filename=file://$(find rebel_arm_description)/meshes/link_6.dae scale=0.001 0.001 0.001
